Commit message: Small update

File: pg70.urdf.xacro (robot description, xacro)
@@ -34,5 +34,6 @@
       <parent link="schunk_palm_link" />
       <child link = "moving_part1" />
-      <origin xyz="0.0 0.0 0.416" rpy="0.0 0.0 0.0" />
+      <origin xyz="0.01 0.01 0.09" rpy="1.57 0.0 0.0" />
+          <limit effort="1000.0" lower="-0.38" upper="0" velocity="0.5"/>
     </joint>
 <link name="right_finger">
@@ -51,5 +52,5 @@
       <parent link="moving_part1" />
       <child link = "right_finger" />
-      <origin xyz="0.0 0.0 0.416" rpy="0.0 0.0 0.0" />
+      <origin xyz="0.0 0.01 0.01" rpy="0.0 0.0 1.57" />
     </joint>
 <link name="moving_part2">
@@ -68,5 +69,6 @@
       <parent link="schunk_palm_link" />
       <child link = "moving_part2" />
-      <origin xyz="0.0 0.0 0.416" rpy="0.0 0.0 0.0" />
+          <limit effort="1000.0" lower="-0.38" upper="0" velocity="0.5"/>
+      <origin xyz="-0.01 -0.01 0.09" rpy="0.0 0.0 0.0" />
     </joint>
 <link name="left_finger">
@@ -85,6 +87,12 @@
       <parent link="moving_part2" />
       <child link = "left_finger" />
-      <origin xyz="0.133 0.0 0.416" rpy="0.0 0.0 0.0" />
+      <origin xyz="0. -0.01 0.01" rpy="0.0 0.0 0.0" />
     </joint>
+<plugin filename="libroboticsgroup_gazebo_mimic_joint_plugin.so" name="mimic_schunk">
+                <joint>moving_part2_joint</joint>
+                <mimicJoint>moving_part1_joint</mimicJoint>
+                <!--multiplier>1.0</multiplier>
+                <offset>0.0</offset-->
+</plugin>
   </xacro:macro>
 </robot>

Commit message: Model created but mimic functionality needs to added

File: pg70.urdf.xacro (robot description, xacro)
@@ -40,10 +40,10 @@
       <visual>
          <geometry>
-          <mesh filename="package://schunk_description/meshes/finger.stl" scale="0.01 0.01 0.01"/>
+          <mesh filename="package://schunk_description/meshes/finger1.dae"/>
         </geometry>
       </visual>
       <collision>
         <geometry>
-          <mesh filename="package://schunk_description/meshes/finger.stl" scale="0.01 0.01 0.01"/>
+          <mesh filename="package://schunk_description/meshes/finger1.dae"/>
         </geometry>
       </collision>
@@ -52,5 +52,5 @@
       <parent link="moving_part1" />
       <child link = "right_finger" />
-      <origin xyz="0.0 0.01 0.01" rpy="0.0 0.0 1.57" />
+      <origin xyz="-0.03 0.06 0.01" rpy="-1.57 0.0 0" />
     </joint>
 <link name="moving_part2">
@@ -75,10 +75,10 @@
       <visual>
          <geometry>
-          <mesh filename="package://schunk_description/meshes/left_finger.stl" scale="0.01 0.01 0.01"/>
+          <mesh filename="package://schunk_description/meshes/finger2.dae" />
         </geometry>
       </visual>
       <collision>
         <geometry>
-          <mesh filename="package://schunk_description/meshes/left_finger.stl" scale="0.01 0.01 0.01"/>
+          <mesh filename="package://schunk_description/meshes/finger2.dae" />
         </geometry>
       </collision>
@@ -87,5 +87,5 @@
       <parent link="moving_part2" />
       <child link = "left_finger" />
-      <origin xyz="0. -0.01 0.01" rpy="0.0 0.0 0.0" />
+      <origin xyz="0.03 0.01 0.06" rpy="0.0 0.0 0.0" />
     </joint>
 <plugin filename="libroboticsgroup_gazebo_mimic_joint_plugin.so" name="mimic_schunk">
